Commit message: Fix ME6 Gazebo world link duplication

File: Homework-3/ros2_ws/src/DOBOT_6Axis_ROS2_V4/cra_description/urdf/me6_robot.xacro (robot description, xacro)
@@ -208,9 +208,4 @@
         <limit lower="-6.27" upper="6.27" effort="300" velocity="300" />
     </joint>
-   <link name="world" />
-    <joint name="world_joint" type="fixed">
-        <parent link="world" />
-        <child link="dummy_link" />
-    </joint>
 <gazebo reference="base_link">
         <gravity>false</gravity>

Commit message: Use official ME6 model for simulation controls

File: Homework-3/ros2_ws/src/DOBOT_6Axis_ROS2_V4/cra_description/urdf/me6_robot.xacro (robot description, xacro)
@@ -1,4 +1,6 @@
 <?xml version="1.0" ?>
 <robot name="me6_robot" xmlns:xacro="http://www.ros.org/wiki/xacro">
+    <xacro:arg name="control_mode" default="gazebo"/>
+    <xacro:property name="control_mode_value" value="$(arg control_mode)"/>
     <link name="dummy_link" />
     <link name="base_link">
@@ -237,8 +239,15 @@
     </gazebo>
     <!-- 在运行demo.launch.py时，需要注释这个ros2_control节点，因为它使用了xxx.ros2_control.xacro来生成了ros2_control节点-->
-    <ros2_control name="GazeboSystem" type="system">
-        <hardware>
-            <plugin>gazebo_ros2_control/GazeboSystem</plugin>
-        </hardware>
+    <ros2_control name="DobotME6System" type="system">
+        <xacro:if value="${control_mode_value == 'gazebo'}">
+            <hardware>
+                <plugin>gazebo_ros2_control/GazeboSystem</plugin>
+            </hardware>
+        </xacro:if>
+        <xacro:if value="${control_mode_value != 'gazebo'}">
+            <hardware>
+                <plugin>fake_components/GenericSystem</plugin>
+            </hardware>
+        </xacro:if>
         <joint name="joint1">
             <command_interface name="position">
@@ -302,9 +311,11 @@
         </joint>
     </ros2_control>
-    <gazebo>
-        <plugin filename="libgazebo_ros2_control.so" name="gazebo_ros2_control">
-            <parameters> $(find me6_moveit)/config/ros2_controllers.yaml</parameters>
-            <robot_param_node>robot_state_publisher</robot_param_node>
-        </plugin>
-    </gazebo>
+    <xacro:if value="${control_mode_value == 'gazebo'}">
+        <gazebo>
+            <plugin filename="libgazebo_ros2_control.so" name="gazebo_ros2_control">
+                <parameters>$(find dobot_me6_bringup)/config/ros2_controllers.yaml</parameters>
+                <robot_param_node>robot_state_publisher</robot_param_node>
+            </plugin>
+        </gazebo>
+    </xacro:if>
 </robot>

Commit message: Show ME6 end-effector position markers

File: Homework-3/ros2_ws/src/DOBOT_6Axis_ROS2_V4/cra_description/urdf/me6_robot.xacro (robot description, xacro)
@@ -210,4 +210,25 @@
         <limit lower="-6.27" upper="6.27" effort="300" velocity="300" />
     </joint>
+    <link name="ee_marker">
+        <inertial>
+            <origin xyz="0 0 0" rpy="0 0 0" />
+            <mass value="0.001" />
+            <inertia ixx="1e-6" ixy="0" ixz="0" iyy="1e-6" iyz="0" izz="1e-6" />
+        </inertial>
+        <visual>
+            <origin xyz="0 0 0" rpy="0 0 0" />
+            <geometry>
+                <sphere radius="0.025" />
+            </geometry>
+            <material name="ee_marker_green">
+                <color rgba="0.0 1.0 0.25 1.0" />
+            </material>
+        </visual>
+    </link>
+    <joint name="ee_marker_fixed" type="fixed">
+        <parent link="Link6" />
+        <child link="ee_marker" />
+        <origin xyz="0 0 0" rpy="0 0 0" />
+    </joint>
 <gazebo reference="base_link">
         <gravity>false</gravity>
@@ -237,4 +258,9 @@
         <gravity>false</gravity>
         <selfCollide>true</selfCollide>
+    </gazebo>
+    <gazebo reference="ee_marker">
+        <material>Gazebo/Green</material>
+        <gravity>false</gravity>
+        <selfCollide>false</selfCollide>
     </gazebo>
     <!-- 在运行demo.launch.py时，需要注释这个ros2_control节点，因为它使用了xxx.ros2_control.xacro来生成了ros2_control节点-->
